Commit message: include package rename ur_picking -> ur_setup_bringup

File: urdf/camera_bracket_adapter.urdf.xacro (robot description, xacro)
@@ -11,5 +11,5 @@
         <origin xyz="0 0 0" rpy="${-pi/2} ${-pi/2} ${pi}"/>
         <geometry>
-          <mesh filename="package://ur_picking/meshes/bracket/ur_D435i_BRACKET.STL" scale="1.0 1.0 1.0"/>
+          <mesh filename="package://ur_setup_bringup/meshes/bracket/ur_D435i_BRACKET.STL" scale="1.0 1.0 1.0"/>
         </geometry>
         <material name="bracket_black">
@@ -20,5 +20,5 @@
         <origin xyz="0 0 0" rpy="${-pi/2} ${-pi/2} ${pi}"/>
         <geometry>
-          <mesh filename="package://ur_picking/meshes/bracket/ur_D435i_BRACKET.STL" scale="1.0 1.0 1.0"/>
+          <mesh filename="package://ur_setup_bringup/meshes/bracket/ur_D435i_BRACKET.STL" scale="1.0 1.0 1.0"/>
         </geometry>
       </collision>

File: urdf/ur16e_robotiq_2f85.urdf.xacro (robot description, xacro)
@@ -26,8 +26,8 @@
        ================================================================ -->
   <xacro:include filename="$(find ur_description)/urdf/ur_macro.xacro"/>
-  <xacro:include filename="$(find ur_picking)/urdf/ur_to_robotiq_adapter.urdf.xacro"/>
+  <xacro:include filename="$(find ur_setup_bringup)/urdf/ur_to_robotiq_adapter.urdf.xacro"/>
   <xacro:include filename="$(find robotiq_description)/urdf/robotiq_2f_85_macro.urdf.xacro"/>
   <!-- 테스트베드 (페데스탈 + 플레이트) 매크로 포함 -->
-  <xacro:include filename="$(find ur_picking)/urdf/testbed.urdf.xacro"/>
+  <xacro:include filename="$(find ur_setup_bringup)/urdf/testbed.urdf.xacro"/>
   <!-- ================================================================
        UR 로봇 기본 인수
@@ -77,7 +77,7 @@
   <xacro:arg name="sim_ignition"           default="false"/>
   <xacro:arg name="simulation_controllers" default=""/>
-  <!-- 초기 자세 (ur_picking 패키지의 공통 파일 사용) -->
+  <!-- 초기 자세 (ur_setup_bringup 패키지의 공통 파일 사용) -->
   <xacro:arg name="initial_positions_file"
-    default="$(find ur_picking)/config/initial_positions.yaml"/>
+    default="$(find ur_setup_bringup)/config/initial_positions.yaml"/>
   <!-- ================================================================
        테스트베드 치수 인수

File: urdf/ur5e_robotiq_2f85.urdf.xacro (robot description, xacro)
@@ -11,9 +11,9 @@
   <xacro:include filename="$(find ur_description)/urdf/ur_macro.xacro"/>
   <!-- 카메라 브라켓 어댑터 -->
-  <xacro:include filename="$(find ur_picking)/urdf/camera_bracket_adapter.urdf.xacro" />
+  <xacro:include filename="$(find ur_setup_bringup)/urdf/camera_bracket_adapter.urdf.xacro" />
   <!-- RealSense D435i 공식 매크로 -->
   <xacro:include filename="$(find realsense2_description)/urdf/_d435i.urdf.xacro" />
   <!-- Use local adapter to avoid duplicate gripper base link -->
-  <xacro:include filename="$(find ur_picking)/urdf/ur_to_robotiq_adapter.urdf.xacro" />
+  <xacro:include filename="$(find ur_setup_bringup)/urdf/ur_to_robotiq_adapter.urdf.xacro" />
   <xacro:include filename="$(find robotiq_description)/urdf/robotiq_2f_85_macro.urdf.xacro" />
   <!-- possible 'ur_type' values: ur3, ur5, ur10, ur3e, ur5e, ur7e, ur10e, ur12e, ur16e, ur8long, ur15, ur18, ur20, ur30 -->
@@ -26,8 +26,8 @@
   <xacro:arg name="physical_params" default="$(find ur_picking)/config/ur5e/physical_parameters.yaml"/>
   <xacro:arg name="visual_params" default="$(find ur_picking)/config/ur5e/visual_parameters.yaml"/> -->
-  <xacro:arg name="joint_limit_params" default="$(find-pkg-share ur_picking)/config/ur5e/joint_limits.yaml"/>
-  <xacro:arg name="kinematics_params" default="$(find-pkg-share ur_picking)/config/ur5e/default_kinematics.yaml"/>
-  <xacro:arg name="physical_params" default="$(find-pkg-share ur_picking)/config/ur5e/physical_parameters.yaml"/>
-  <xacro:arg name="visual_params" default="$(find-pkg-share ur_picking)/config/ur5e/visual_parameters.yaml"/>
+  <xacro:arg name="joint_limit_params" default="$(find-pkg-share ur_setup_bring)/config/ur5e/joint_limits.yaml"/>
+  <xacro:arg name="kinematics_params" default="$(find-pkg-share ur_setup_bring)/config/ur5e/default_kinematics.yaml"/>
+  <xacro:arg name="physical_params" default="$(find-pkg-share ur_setup_bring)/config/ur5e/physical_parameters.yaml"/>
+  <xacro:arg name="visual_params" default="$(find-pkg-share ur_setup_bring)/config/ur5e/visual_parameters.yaml"/>
   <xacro:arg name="transmission_hw_interface" default=""/>
   <xacro:arg name="safety_limits" default="false"/>
