Commit message: 1. 알파벳EDGE BRAIN 추가 - 가제보 스폰방식, 2. 가제보 테스트베드 디지털트윈

File: urdf/testbed.urdf.xacro (robot description, xacro)
@@ -13,14 +13,18 @@
       pedestal_x      : 페데스탈 X 방향 길이 [m] (기본: 1.2)
       pedestal_y      : 페데스탈 Y 방향 폭   [m] (기본: 0.6)
-      pedestal_z      : 페데스탈 높이         [m] (기본: 0.8)
+      pedestal_z      : 페데스탈 높이         [m] (기본: 0.9)
       pedestal_mass   : 페데스탈 질량         [kg] (기본: 150.0)
-      plate_size_x    : 플레이트 X 방향 길이  [m] (기본: 0.4)
-      plate_size_y    : 플레이트 Y 방향 폭    [m] (기본: 0.4)
+      plate_size_x    : 좌측 plate X 방향 길이 [m] (기본: 0.6)
+      plate_size_y    : 좌측 plate Y 방향 폭   [m] (기본: 0.6)
       plate_thickness : 플레이트 두께         [m] (기본: 0.02)
-      plate_mass      : 플레이트 1개 질량     [kg] (기본: 8.6)
-      plate_left_x    : 좌측 플레이트 중심 X  [m, robot base 프레임 기준] (기본: 0.45)
-      plate_left_y    : 좌측 플레이트 중심 Y  [m, robot base 프레임 기준] (기본: 0.35)
-      plate_right_x   : 우측 플레이트 중심 X  [m, robot base 프레임 기준] (기본: 0.45)
-      plate_right_y   : 우측 플레이트 중심 Y  [m, robot base 프레임 기준] (기본: -0.35)
+      plate_mass      : 좌측 plate 질량        [kg] (기본: 8.6)
+      pallet_size_x   : 우측 pallet X 방향 길이 [m] (기본: 0.6)
+      pallet_size_y   : 우측 pallet Y 방향 폭   [m] (기본: 0.35)
+      pallet_thickness: 우측 pallet 두께        [m] (기본: 0.02)
+      pallet_mass     : 우측 pallet 질량        [kg] (기본: 8.6)
+      plate_x         : 좌측 plate 중심 X  [m, robot base 프레임 기준] (기본: 0.45)
+      plate_y         : 좌측 plate 중심 Y  [m, robot base 프레임 기준] (기본: 0.35)
+      pallet_x        : 우측 pallet 중심 X [m, robot base 프레임 기준] (기본: -0.45)
+      pallet_y        : 우측 pallet 중심 Y [m, robot base 프레임 기준] (기본: 0.35)
       obstacle_*      : 선택적 고정 충돌 직육면체
                         기본은 비활성화. command 기반 spawn/remove 사용 권장.
@@ -29,16 +33,20 @@
     params="
       parent:=world
-      pedestal_x:=1.8
-      pedestal_y:=1.0
-      pedestal_z:=0.8
+      pedestal_x:=2.0
+      pedestal_y:=0.8
+      pedestal_z:=0.9
       pedestal_mass:=150.0
-      plate_size_x:=0.4
-      plate_size_y:=0.4
+      plate_size_x:=0.6
+      plate_size_y:=0.6
       plate_thickness:=0.02
+      pallet_size_x:=0.6
+      pallet_size_y:=0.35
+      pallet_thickness:=0.02
+      pallet_mass:=8.6
       plate_mass:=8.6
-      plate_left_x:=0.45
-      plate_left_y:=0.35
-      plate_right_x:=-0.45
-      plate_right_y:=0.35
+      plate_x:=0.60
+      plate_y:=0.25
+      pallet_x:=-0.60
+      pallet_y:=0.35
       obstacle_enabled:=false
       obstacle_x:=0.0
@@ -46,5 +54,5 @@
       obstacle_size_x:=0.05
       obstacle_size_y:=0.30
-      obstacle_size_z:=0.40
+      obstacle_size_z:=0.30
       obstacle_mass:=3.0">
     <!-- ==============================================================
@@ -101,6 +109,6 @@
     <!-- ==============================================================
          좌측 작업 플레이트 (plate_left_link)
-         world 프레임 좌표: (plate_left_x, plate_left_y, pedestal_z + plate_thickness/2)
-         robot base 프레임 좌표: (plate_left_x, plate_left_y, plate_thickness/2)
+         world 프레임 좌표: (plate_x, plate_y, pedestal_z + plate_thickness/2)
+         robot base 프레임 좌표: (plate_x, plate_y, plate_thickness/2)
          ============================================================== -->
     <link name="plate_left_link">
@@ -110,6 +118,6 @@
           <box size="${plate_size_x} ${plate_size_y} ${plate_thickness}"/>
         </geometry>
-        <material name="plate_aluminum">
-          <color rgba="0.78 0.78 0.78 1.0"/>
+        <material name="plate_green">
+          <color rgba="0.10 0.65 0.18 1.0"/>
         </material>
       </visual>
@@ -142,10 +150,10 @@
       <child link="plate_left_link"/>
       <origin
-        xyz="${plate_left_x} ${plate_left_y} ${pedestal_z + plate_thickness/2}"
+        xyz="${plate_x} ${plate_y} ${pedestal_z + plate_thickness/2}"
         rpy="0 0 0"/>
     </joint>
-    <!-- Gazebo 재질: 밝은 회색, 블록 안착을 위한 마찰 계수 -->
+    <!-- Gazebo 재질: green, 블록 안착을 위한 마찰 계수 -->
     <gazebo reference="plate_left_link">
-      <material>Gazebo/Grey</material>
+      <material>Gazebo/Green</material>
       <mu1>0.8</mu1>
       <mu2>0.8</mu2>
@@ -153,5 +161,5 @@
     </gazebo>
     <!-- ==============================================================
-         우측 작업 플레이트 (plate_right_link)
+         우측 팔레트 (plate_right_link)
          ============================================================== -->
     <link name="plate_right_link">
@@ -159,8 +167,8 @@
         <origin xyz="0 0 0" rpy="0 0 0"/>
         <geometry>
-          <box size="${plate_size_x} ${plate_size_y} ${plate_thickness}"/>
-        </geometry>
-        <material name="plate_aluminum">
-          <color rgba="0.78 0.78 0.78 1.0"/>
+          <box size="${pallet_size_x} ${pallet_size_y} ${pallet_thickness}"/>
+        </geometry>
+        <material name="pallet_blue">
+          <color rgba="0.05 0.25 0.90 1.0"/>
         </material>
       </visual>
@@ -168,16 +176,16 @@
         <origin xyz="0 0 0" rpy="0 0 0"/>
         <geometry>
-          <box size="${plate_size_x} ${plate_size_y} ${plate_thickness}"/>
+          <box size="${pallet_size_x} ${pallet_size_y} ${pallet_thickness}"/>
         </geometry>
       </collision>
       <inertial>
-        <mass value="${plate_mass}"/>
+        <mass value="${pallet_mass}"/>
         <origin xyz="0 0 0" rpy="0 0 0"/>
         <inertia
-          ixx="${(1.0/12.0) * plate_mass * (plate_size_y**2 + plate_thickness**2)}"
+          ixx="${(1.0/12.0) * pallet_mass * (pallet_size_y**2 + pallet_thickness**2)}"
           ixy="0" ixz="0"
-          iyy="${(1.0/12.0) * plate_mass * (plate_size_x**2 + plate_thickness**2)}"
+          iyy="${(1.0/12.0) * pallet_mass * (pallet_size_x**2 + pallet_thickness**2)}"
           iyz="0"
-          izz="${(1.0/12.0) * plate_mass * (plate_size_x**2 + plate_size_y**2)}"/>
+          izz="${(1.0/12.0) * pallet_mass * (pallet_size_x**2 + pallet_size_y**2)}"/>
       </inertial>
     </link>
@@ -186,9 +194,9 @@
       <child link="plate_right_link"/>
       <origin
-        xyz="${plate_right_x} ${plate_right_y} ${pedestal_z + plate_thickness/2}"
+        xyz="${pallet_x} ${pallet_y} ${pedestal_z + pallet_thickness/2}"
         rpy="0 0 0"/>
     </joint>
     <gazebo reference="plate_right_link">
-      <material>Gazebo/Grey</material>
+      <material>Gazebo/Blue</material>
       <mu1>0.8</mu1>
       <mu2>0.8</mu2>

File: urdf/ur16e_robotiq_2f85.urdf.xacro (robot description, xacro)
@@ -91,5 +91,5 @@
        변경 시 testbed.urdf.xacro 의 params 블록만 수정하면 됨.
        ================================================================ -->
-  <xacro:arg name="pedestal_z" default="0.8"/>
+  <xacro:arg name="pedestal_z" default="0.9"/>
   <!-- xacro 표현식에서 사용하기 위해 property 로 변환 -->
   <xacro:property name="initial_positions_file" value="$(arg initial_positions_file)"/>
