Commit message: RTF가 0.2로 떨어짐에 따라서, 다음 수정사항을 적용. -> 1. 시뮬레이션 update_rate 감소 2. attach를 위한 plugin 작성

File: urdf/ur16e_robotiq_2f85.urdf.xacro (robot description, xacro)
@@ -195,5 +195,5 @@
       </camera>
       <always_on>1</always_on>
-      <update_rate>30</update_rate>
+      <update_rate>1</update_rate>
       <visualize>true</visualize>
       <topic>$(arg tf_prefix)camera</topic>
@@ -231,4 +231,46 @@
       </plugin>
     </gazebo>
+    <!-- ================================================================
+         DetachableJoint 플러그인 (alphabet 잡기 RTF 회복용)
+         pick 직후 dispatcher 가 /grasp/attach/<letter> 에 publish 하면
+         해당 alphabet 이 tool0 와 fixed joint 로 묶여 contact 해석을 우회.
+         place 직전 pick_place_node 가 /grasp/release_all 에 publish 하여
+         모든 attached letter 를 detach (한 번에 풀어도 안전, idempotent).
+         설계 메모:
+           parent_link 는 URDF/SDF 변환에서 살아남는 링크여야 함.
+           robotiq_85_base_link 같은 adapter 하위 링크는 fixed joint
+           collapse 로 사라질 수 있으므로 표준 UR 링크 tool0 사용.
+           9개 인스턴스를 별도 <gazebo> 블록으로 분리 (SDF 파서 안전).
+           시작 시 isAttached=false (소스 확인) 라 명시 attach 전엔 dormant.
+         ================================================================ -->
+    <xacro:macro name="alphabet_attach_plugin" params="model_name">
+      <gazebo>
+        <plugin
+          filename="ignition-gazebo-detachable-joint-system"
+          name="ignition::gazebo::systems::DetachableJoint">
+          <!-- 주의: tool0, robotiq_85_base_link 등은 URDF→SDF 변환 시 fixed
+               joint 가 부모로 collapse 되어 사라짐. wrist_3_link 는 UR arm
+               의 마지막 revolute link 라 항상 살아있고 gripper 위에 고정.
+               attach 시점의 wrist_3_link ↔ letter 상대 pose 가 joint 로 잠김. -->
+          <parent_link>$(arg tf_prefix)wrist_3_link</parent_link>
+          <child_model>${model_name}</child_model>
+          <child_link>link</child_link>
+          <attach_topic>/grasp/attach/${model_name}</attach_topic>
+          <detach_topic>/grasp/release_all</detach_topic>
+          <output_topic>/grasp/state/${model_name}</output_topic>
+          <suppress_child_warning>true</suppress_child_warning>
+        </plugin>
+      </gazebo>
+    </xacro:macro>
+    <!-- launch/dispatcher 의 EDGE BRAIN sequence 순서와 동일하게 정렬 -->
+    <xacro:alphabet_attach_plugin model_name="alphabet_E1"/>
+    <xacro:alphabet_attach_plugin model_name="alphabet_D"/>
+    <xacro:alphabet_attach_plugin model_name="alphabet_G"/>
+    <xacro:alphabet_attach_plugin model_name="alphabet_E2"/>
+    <xacro:alphabet_attach_plugin model_name="alphabet_B"/>
+    <xacro:alphabet_attach_plugin model_name="alphabet_R"/>
+    <xacro:alphabet_attach_plugin model_name="alphabet_A"/>
+    <xacro:alphabet_attach_plugin model_name="alphabet_I"/>
+    <xacro:alphabet_attach_plugin model_name="alphabet_N"/>
   </xacro:if>
   <xacro:if value="$(arg sim_gazebo)">

Commit message: Add OpenVLA UR16e simulation setting - delete wrist camera, create color blocks, 3rd camera

File: urdf/ur16e_robotiq_2f85.urdf.xacro (robot description, xacro)
@@ -92,4 +92,11 @@
        ================================================================ -->
   <xacro:arg name="pedestal_z" default="0.9"/>
+  <xacro:arg name="enable_third_person_camera" default="false"/>
+  <xacro:arg name="openvla_camera_x" default="1.80"/>
+  <xacro:arg name="openvla_camera_y" default="-1.90"/>
+  <xacro:arg name="openvla_camera_z" default="2.90"/>
+  <xacro:arg name="openvla_camera_roll" default="0.0"/>
+  <xacro:arg name="openvla_camera_pitch" default="0.58"/>
+  <xacro:arg name="openvla_camera_yaw" default="2.25"/>
   <!-- xacro 표현식에서 사용하기 위해 property 로 변환 -->
   <xacro:property name="initial_positions_file" value="$(arg initial_positions_file)"/>
@@ -160,45 +167,94 @@
     prefix="$(arg tf_prefix)"
     parent="$(arg tf_prefix)tool0"/>
-  <xacro:sensor_d435
-    parent="$(arg tf_prefix)camera_mounting_point"
-    name="$(arg tf_prefix)camera"
-    use_nominal_extrinsics="true">
-    <origin xyz="0 0 0" rpy="0 0 0"/>
-  </xacro:sensor_d435>
   <!--
-    Ignition Gazebo RGBD 카메라 센서 플러그인.
-    - type="rgbd_camera": 컬러 이미지 + 뎁스 이미지 + 포인트 클라우드를 동시에 발행
-    - reference: sensor_d435 매크로가 생성하는 camera_link 프레임을 참조
-    - topic: Ignition 내부 토픽 prefix (ros_gz_bridge에서 ROS2 토픽으로 변환)
-    - ignition_frame_id: 발행되는 이미지 메시지의 frame_id (Fortress 전용 태그, gz_frame_id는 Garden+에서만 유효)
-    - sensors 시스템 플러그인은 world SDF(testbed.sdf)에서 로드됨
+    Wrist RealSense D435 disabled for OpenVLA third-person experiments.
+    To restore it later, change the xacro:if value below from "false" to "true".
+    Keep camera_bracket_adapter above enabled because it also provides the gripper mount.
   -->
-  <gazebo reference="$(arg tf_prefix)camera_link">
-    <sensor name="$(arg tf_prefix)d435_rgbd" type="rgbd_camera">
-      <camera>
-        <!-- D435 수평 시야각: 약 86도 = 1.5009 rad -->
-        <horizontal_fov>1.5009</horizontal_fov>
-        <image>
-          <width>848</width>
-          <height>480</height>
-          <format>R8G8B8</format>
-        </image>
-        <clip>
-          <near>0.105</near>
-          <far>10.0</far>
-        </clip>
-        <noise>
-          <type>gaussian</type>
-          <mean>0.0</mean>
-          <stddev>0.007</stddev>
-        </noise>
-      </camera>
-      <always_on>1</always_on>
-      <update_rate>1</update_rate>
-      <visualize>true</visualize>
-      <topic>$(arg tf_prefix)camera</topic>
-      <ignition_frame_id>$(arg tf_prefix)camera_color_optical_frame</ignition_frame_id>
-    </sensor>
-  </gazebo>
+  <xacro:if value="false">
+    <xacro:sensor_d435
+      parent="$(arg tf_prefix)camera_mounting_point"
+      name="$(arg tf_prefix)camera"
+      use_nominal_extrinsics="true">
+      <origin xyz="0 0 0" rpy="0 0 0"/>
+    </xacro:sensor_d435>
+    <!--
+      Ignition Gazebo RGBD 카메라 센서 플러그인.
+      - type="rgbd_camera": 컬러 이미지 + 뎁스 이미지 + 포인트 클라우드를 동시에 발행
+      - reference: sensor_d435 매크로가 생성하는 camera_link 프레임을 참조
+      - topic: Ignition 내부 토픽 prefix (ros_gz_bridge에서 ROS2 토픽으로 변환)
+      - ignition_frame_id: 발행되는 이미지 메시지의 frame_id (Fortress 전용 태그, gz_frame_id는 Garden+에서만 유효)
+      - sensors 시스템 플러그인은 world SDF(testbed.sdf)에서 로드됨
+    -->
+    <gazebo reference="$(arg tf_prefix)camera_link">
+      <sensor name="$(arg tf_prefix)d435_rgbd" type="rgbd_camera">
+        <camera>
+          <!-- D435 수평 시야각: 약 86도 = 1.5009 rad -->
+          <horizontal_fov>1.5009</horizontal_fov>
+          <image>
+            <width>848</width>
+            <height>480</height>
+            <format>R8G8B8</format>
+          </image>
+          <clip>
+            <near>0.105</near>
+            <far>10.0</far>
+          </clip>
+          <noise>
+            <type>gaussian</type>
+            <mean>0.0</mean>
+            <stddev>0.007</stddev>
+          </noise>
+        </camera>
+        <always_on>1</always_on>
+        <update_rate>1</update_rate>
+        <visualize>true</visualize>
+        <topic>$(arg tf_prefix)camera</topic>
+        <ignition_frame_id>$(arg tf_prefix)camera_color_optical_frame</ignition_frame_id>
+      </sensor>
+    </gazebo>
+  </xacro:if>
+  <!-- ================================================================
+       OpenVLA 입력용 third-person RealSense D435 RGBD camera
+       - world 에 fixed joint 로 연결되어 RViz RobotModel / TF 에서 위치 확인 가능
+       - D435 mesh 를 사용하되 rgbd_camera sensor 로 depth / point cloud 도 발행
+       ================================================================ -->
+  <xacro:if value="$(arg enable_third_person_camera)">
+    <xacro:sensor_d435
+      parent="world"
+      name="openvla_camera"
+      use_nominal_extrinsics="true">
+      <origin
+        xyz="$(arg openvla_camera_x) $(arg openvla_camera_y) $(arg openvla_camera_z)"
+        rpy="$(arg openvla_camera_roll) $(arg openvla_camera_pitch) $(arg openvla_camera_yaw)"/>
+    </xacro:sensor_d435>
+    <gazebo reference="openvla_camera_link">
+      <sensor name="openvla_camera_d435_rgbd" type="rgbd_camera">
+        <camera>
+          <!-- D435 수평 시야각: 약 86도 = 1.5009 rad -->
+          <horizontal_fov>1.5009</horizontal_fov>
+          <image>
+            <width>848</width>
+            <height>480</height>
+            <format>R8G8B8</format>
+          </image>
+          <clip>
+            <near>0.105</near>
+            <far>10.0</far>
+          </clip>
+          <noise>
+            <type>gaussian</type>
+            <mean>0.0</mean>
+            <stddev>0.007</stddev>
+          </noise>
+        </camera>
+        <always_on>1</always_on>
+        <update_rate>10</update_rate>
+        <visualize>true</visualize>
+        <topic>openvla_camera</topic>
+        <ignition_frame_id>openvla_camera_color_optical_frame</ignition_frame_id>
+      </sensor>
+    </gazebo>
+  </xacro:if>
   <!-- ================================================================
        Robotiq 2F-85 어댑터 + 그리퍼 (브라켓의 gripper_mounting_point 기준)

Commit message: 블록 생성으로 수정

File: urdf/ur16e_robotiq_2f85.urdf.xacro (robot description, xacro)
@@ -288,7 +288,8 @@
     </gazebo>
     <!-- ================================================================
-         DetachableJoint 플러그인 (alphabet 잡기 RTF 회복용)
-         pick 직후 dispatcher 가 /grasp/attach/<letter> 에 publish 하면
-         해당 alphabet 이 tool0 와 fixed joint 로 묶여 contact 해석을 우회.
+         DetachableJoint 플러그인 (grasp 후 contact/collision 해석 회피용)
+         pick 직후 dispatcher/episode runner 가 /grasp/attach/<object> 에
+         publish 하면 해당 object 가 tool0 와 fixed joint 로 묶여 contact
+         해석을 우회.
          place 직전 pick_place_node 가 /grasp/release_all 에 publish 하여
          모든 attached letter 를 detach (한 번에 풀어도 안전, idempotent).
@@ -300,5 +301,5 @@
            시작 시 isAttached=false (소스 확인) 라 명시 attach 전엔 dormant.
          ================================================================ -->
-    <xacro:macro name="alphabet_attach_plugin" params="model_name">
+    <xacro:macro name="detachable_joint_plugin" params="model_name">
       <gazebo>
         <plugin
@@ -320,13 +321,16 @@
     </xacro:macro>
     <!-- launch/dispatcher 의 EDGE BRAIN sequence 순서와 동일하게 정렬 -->
-    <xacro:alphabet_attach_plugin model_name="alphabet_E1"/>
-    <xacro:alphabet_attach_plugin model_name="alphabet_D"/>
-    <xacro:alphabet_attach_plugin model_name="alphabet_G"/>
-    <xacro:alphabet_attach_plugin model_name="alphabet_E2"/>
-    <xacro:alphabet_attach_plugin model_name="alphabet_B"/>
-    <xacro:alphabet_attach_plugin model_name="alphabet_R"/>
-    <xacro:alphabet_attach_plugin model_name="alphabet_A"/>
-    <xacro:alphabet_attach_plugin model_name="alphabet_I"/>
-    <xacro:alphabet_attach_plugin model_name="alphabet_N"/>
+    <xacro:detachable_joint_plugin model_name="alphabet_E1"/>
+    <xacro:detachable_joint_plugin model_name="alphabet_D"/>
+    <xacro:detachable_joint_plugin model_name="alphabet_G"/>
+    <xacro:detachable_joint_plugin model_name="alphabet_E2"/>
+    <xacro:detachable_joint_plugin model_name="alphabet_B"/>
+    <xacro:detachable_joint_plugin model_name="alphabet_R"/>
+    <xacro:detachable_joint_plugin model_name="alphabet_A"/>
+    <xacro:detachable_joint_plugin model_name="alphabet_I"/>
+    <xacro:detachable_joint_plugin model_name="alphabet_N"/>
+    <!-- OpenVLA colored-block episode targets. -->
+    <xacro:detachable_joint_plugin model_name="block_red"/>
+    <xacro:detachable_joint_plugin model_name="block_yellow"/>
   </xacro:if>
   <xacro:if value="$(arg sim_gazebo)">
