Commit message: modified camera pose

File: srdf/ur_robotiq.srdf.xacro (robot description, xacro)
@@ -154,8 +154,5 @@
   <disable_collisions link1="$(arg prefix)camera_infra2_frame" link2="$(arg prefix)camera_depth_frame" reason="Adjacent" />
   <disable_collisions link1="$(arg prefix)camera_infra2_optical_frame" link2="$(arg prefix)camera_infra2_frame" reason="Adjacent" />
-  <disable_collisions link1="$(arg prefix)camera_accel_frame" link2="$(arg prefix)camera_link" reason="Adjacent" />
-  <disable_collisions link1="$(arg prefix)camera_accel_optical_frame" link2="$(arg prefix)camera_accel_frame" reason="Adjacent" />
-  <disable_collisions link1="$(arg prefix)camera_gyro_frame" link2="$(arg prefix)camera_link" reason="Adjacent" />
-  <disable_collisions link1="$(arg prefix)camera_gyro_optical_frame" link2="$(arg prefix)camera_gyro_frame" reason="Adjacent" />
+  <!-- D435i 전용 IMU 링크 (camera_accel_*, camera_gyro_*) 는 D435에 존재하지 않으므로 제거 -->
     <!-- ================================================================
        테스트베드 환경 링크 충돌 설정

File: urdf/camera_bracket_adapter.urdf.xacro (robot description, xacro)
@@ -5,5 +5,5 @@
       <parent link="${parent}"/>
       <child link="${prefix}camera_bracket_link"/>
-      <origin xyz="0 0 0" rpy="0 0 0"/>
+      <origin xyz="0 0 0" rpy="0 0 ${pi/2}"/>
     </joint>
     <link name="${prefix}camera_bracket_link">
@@ -39,5 +39,5 @@
       <parent link="${prefix}camera_bracket_link"/>
       <child link="${prefix}gripper_mounting_point"/>
-      <origin xyz="0 0 0.008" rpy="0 0 ${pi/2}"/>
+      <origin xyz="0 0 0.008" rpy="0 0 0"/>
     </joint>
     <link name="${prefix}gripper_mounting_point"/>

File: urdf/ur16e_robotiq_2f85.urdf.xacro (robot description, xacro)
@@ -26,4 +26,8 @@
        ================================================================ -->
   <xacro:include filename="$(find ur_description)/urdf/ur_macro.xacro"/>
+  <!-- 카메라 브라켓 어댑터 (tool0 -> camera_mounting_point + gripper_mounting_point) -->
+  <xacro:include filename="$(find ur_setup_bringup)/urdf/camera_bracket_adapter.urdf.xacro"/>
+  <!-- RealSense D435 (D435i의 IMU 모듈은 Ignition Fortress와 호환 불가) -->
+  <xacro:include filename="$(find realsense2_description)/urdf/_d435.urdf.xacro"/>
   <xacro:include filename="$(find ur_setup_bringup)/urdf/ur_to_robotiq_adapter.urdf.xacro"/>
   <xacro:include filename="$(find robotiq_description)/urdf/robotiq_2f_85_macro.urdf.xacro"/>
@@ -151,9 +155,56 @@
   </xacro:ur_robot>
   <!-- ================================================================
-       Robotiq 2F-85 어댑터 + 그리퍼 (tool0 기준)
+       카메라 브라켓 + RealSense D435 (tool0 기준)
+       ================================================================ -->
+  <xacro:camera_bracket_adapter
+    prefix="$(arg tf_prefix)"
+    parent="$(arg tf_prefix)tool0"/>
+  <xacro:sensor_d435
+    parent="$(arg tf_prefix)camera_mounting_point"
+    name="$(arg tf_prefix)camera"
+    use_nominal_extrinsics="true">
+    <origin xyz="0 0 0" rpy="0 0 0"/>
+  </xacro:sensor_d435>
+  <!--
+    Ignition Gazebo RGBD 카메라 센서 플러그인.
+    - type="rgbd_camera": 컬러 이미지 + 뎁스 이미지 + 포인트 클라우드를 동시에 발행
+    - reference: sensor_d435 매크로가 생성하는 camera_link 프레임을 참조
+    - topic: Ignition 내부 토픽 prefix (ros_gz_bridge에서 ROS2 토픽으로 변환)
+    - ignition_frame_id: 발행되는 이미지 메시지의 frame_id (Fortress 전용 태그, gz_frame_id는 Garden+에서만 유효)
+    - sensors 시스템 플러그인은 world SDF(testbed.sdf)에서 로드됨
+  -->
+  <gazebo reference="$(arg tf_prefix)camera_link">
+    <sensor name="$(arg tf_prefix)d435_rgbd" type="rgbd_camera">
+      <camera>
+        <!-- D435 수평 시야각: 약 86도 = 1.5009 rad -->
+        <horizontal_fov>1.5009</horizontal_fov>
+        <image>
+          <width>848</width>
+          <height>480</height>
+          <format>R8G8B8</format>
+        </image>
+        <clip>
+          <near>0.105</near>
+          <far>10.0</far>
+        </clip>
+        <noise>
+          <type>gaussian</type>
+          <mean>0.0</mean>
+          <stddev>0.007</stddev>
+        </noise>
+      </camera>
+      <always_on>1</always_on>
+      <update_rate>30</update_rate>
+      <visualize>true</visualize>
+      <topic>$(arg tf_prefix)camera</topic>
+      <ignition_frame_id>$(arg tf_prefix)camera_color_optical_frame</ignition_frame_id>
+    </sensor>
+  </gazebo>
+  <!-- ================================================================
+       Robotiq 2F-85 어댑터 + 그리퍼 (브라켓의 gripper_mounting_point 기준)
        ================================================================ -->
   <xacro:ur_to_robotiq
     prefix="$(arg tf_prefix)"
-    parent="$(arg tf_prefix)tool0"
+    parent="$(arg tf_prefix)gripper_mounting_point"
     child="$(arg tf_prefix)robotiq_85_base_link"/>
   <xacro:robotiq_gripper

File: urdf/ur5e_robotiq_2f85.urdf.xacro (robot description, xacro)
@@ -12,6 +12,6 @@
   <!-- 카메라 브라켓 어댑터 -->
   <xacro:include filename="$(find ur_setup_bringup)/urdf/camera_bracket_adapter.urdf.xacro" />
-  <!-- RealSense D435i 공식 매크로 -->
-  <xacro:include filename="$(find realsense2_description)/urdf/_d435i.urdf.xacro" />
+  <!-- RealSense D435 공식 매크로 (D435i의 IMU 모듈은 Ignition Fortress와 호환 불가) -->
+  <xacro:include filename="$(find realsense2_description)/urdf/_d435.urdf.xacro" />
   <!-- Use local adapter to avoid duplicate gripper base link -->
   <xacro:include filename="$(find ur_setup_bringup)/urdf/ur_to_robotiq_adapter.urdf.xacro" />
@@ -64,5 +64,5 @@
   <!-- 로컬 ur_picking 초기자세 사용 -->
   <!-- <xacro:arg name="initial_positions_file" default="$(find ur_picking)/config/initial_positions.yaml"/> -->
-  <xacro:arg name="initial_positions_file" default="$(find-pkg-share ur_picking)/config/initial_positions.yaml"/>
+  <xacro:arg name="initial_positions_file" default="$(find-pkg-share ur_setup_bringup)/config/initial_positions.yaml"/>
   <!-- convert to property to use substitution in function -->
   <xacro:property name="initial_positions_file" default="$(arg initial_positions_file)"/>
@@ -140,11 +140,48 @@
     prefix="$(arg tf_prefix)"
     parent="$(arg tf_prefix)tool0" />
-  <!-- ===================== RealSense D435i 카메라 부착 (브라켓에) ===================== -->
-  <xacro:sensor_d435i
+  <!-- ===================== RealSense D435 카메라 부착 (브라켓에) ===================== -->
+  <xacro:sensor_d435
     parent="$(arg tf_prefix)camera_mounting_point"
     name="$(arg tf_prefix)camera"
     use_nominal_extrinsics="true">
     <origin xyz="0 0 0" rpy="0 0 0"/>
-  </xacro:sensor_d435i>
+  </xacro:sensor_d435>
+  <!--
+    Ignition Gazebo RGBD 카메라 센서 플러그인.
+    - type="rgbd_camera": 컬러 이미지 + 뎁스 이미지 + 포인트 클라우드를 동시에 발행
+    - reference: sensor_d435 매크로가 생성하는 camera_link 프레임을 참조
+    - topic: Ignition 내부 토픽 prefix (ros_gz_bridge에서 ROS2 토픽으로 변환)
+    - ignition_frame_id: 발행되는 이미지 메시지의 frame_id (Fortress 전용 태그, gz_frame_id는 Garden+에서만 유효)
+    - sensors 시스템 플러그인은 world SDF 파일(testbed.sdf / simulation.sdf)에서 로드됨
+  -->
+  <gazebo reference="$(arg tf_prefix)camera_link">
+    <sensor name="$(arg tf_prefix)d435_rgbd" type="rgbd_camera">
+      <camera>
+        <!-- D435 수평 시야각: 약 86도 = 1.5009 rad -->
+        <horizontal_fov>1.5009</horizontal_fov>
+        <image>
+          <width>848</width>
+          <height>480</height>
+          <format>R8G8B8</format>
+        </image>
+        <clip>
+          <near>0.105</near>
+          <far>10.0</far>
+        </clip>
+        <noise>
+          <type>gaussian</type>
+          <mean>0.0</mean>
+          <stddev>0.007</stddev>
+        </noise>
+      </camera>
+      <always_on>1</always_on>
+      <update_rate>30</update_rate>
+      <visualize>true</visualize>
+      <!-- Ignition 내부 토픽 이름 (ros_gz_bridge가 이 이름을 기준으로 브리지함) -->
+      <topic>$(arg tf_prefix)camera</topic>
+      <!-- 발행되는 Image/PointCloud2 메시지의 header.frame_id -->
+      <ignition_frame_id>$(arg tf_prefix)camera_color_optical_frame</ignition_frame_id>
+    </sensor>
+  </gazebo>
   <!-- ===================== Robotiq 2F-85 어댑터 + 그리퍼 부착 (브라켓에) ===================== -->
   <xacro:ur_to_robotiq

Commit message: 수정: kinematics.yaml에서 KDL -> bio_ik로 변경, 초기 위치 변경, obstacle 객체 추가/제거 기능

File: srdf/ur_robotiq.srdf.xacro (robot description, xacro)
@@ -154,5 +154,4 @@
   <disable_collisions link1="$(arg prefix)camera_infra2_frame" link2="$(arg prefix)camera_depth_frame" reason="Adjacent" />
   <disable_collisions link1="$(arg prefix)camera_infra2_optical_frame" link2="$(arg prefix)camera_infra2_frame" reason="Adjacent" />
-  <!-- D435i 전용 IMU 링크 (camera_accel_*, camera_gyro_*) 는 D435에 존재하지 않으므로 제거 -->
     <!-- ================================================================
        테스트베드 환경 링크 충돌 설정

File: urdf/testbed.urdf.xacro (robot description, xacro)
@@ -23,4 +23,6 @@
       plate_right_x   : 우측 플레이트 중심 X  [m, robot base 프레임 기준] (기본: 0.45)
       plate_right_y   : 우측 플레이트 중심 Y  [m, robot base 프레임 기준] (기본: -0.35)
+      obstacle_*      : 선택적 고정 충돌 직육면체
+                        기본은 비활성화. command 기반 spawn/remove 사용 권장.
   -->
   <xacro:macro name="testbed"
@@ -38,5 +40,12 @@
       plate_left_y:=0.35
       plate_right_x:=-0.45
-      plate_right_y:=0.35">
+      plate_right_y:=0.35
+      obstacle_enabled:=false
+      obstacle_x:=0.0
+      obstacle_y:=0.45
+      obstacle_size_x:=0.05
+      obstacle_size_y:=0.30
+      obstacle_size_z:=0.40
+      obstacle_mass:=3.0">
     <!-- ==============================================================
          페데스탈 (받침대)
@@ -186,4 +195,52 @@
       <selfCollide>false</selfCollide>
     </gazebo>
+    <!-- ==============================================================
+         선택적 고정 충돌 직육면체
+         command 기반 Gazebo spawn/remove + PlanningScene add/remove 를
+         사용할 때는 obstacle_enabled=false 상태를 유지한다.
+         필요 시에만 true 로 켜며, 기본 위치는 로봇에서 x=10 m 떨어진 곳.
+         ============================================================== -->
+    <xacro:if value="${obstacle_enabled}">
+      <link name="testbed_obstacle_link">
+        <visual>
+          <origin xyz="0 0 0" rpy="0 0 0"/>
+          <geometry>
+            <box size="${obstacle_size_x} ${obstacle_size_y} ${obstacle_size_z}"/>
+          </geometry>
+          <material name="obstacle_red">
+            <color rgba="0.80 0.10 0.08 1.0"/>
+          </material>
+        </visual>
+        <collision>
+          <origin xyz="0 0 0" rpy="0 0 0"/>
+          <geometry>
+            <box size="${obstacle_size_x} ${obstacle_size_y} ${obstacle_size_z}"/>
+          </geometry>
+        </collision>
+        <inertial>
+          <mass value="${obstacle_mass}"/>
+          <origin xyz="0 0 0" rpy="0 0 0"/>
+          <inertia
+            ixx="${(1.0/12.0) * obstacle_mass * (obstacle_size_y**2 + obstacle_size_z**2)}"
+            ixy="0" ixz="0"
+            iyy="${(1.0/12.0) * obstacle_mass * (obstacle_size_x**2 + obstacle_size_z**2)}"
+            iyz="0"
+            izz="${(1.0/12.0) * obstacle_mass * (obstacle_size_x**2 + obstacle_size_y**2)}"/>
+        </inertial>
+      </link>
+      <joint name="testbed_obstacle_joint" type="fixed">
+        <parent link="${parent}"/>
+        <child link="testbed_obstacle_link"/>
+        <origin
+          xyz="${obstacle_x} ${obstacle_y} ${pedestal_z + obstacle_size_z / 2.0}"
+          rpy="0 0 0"/>
+      </joint>
+      <gazebo reference="testbed_obstacle_link">
+        <material>Gazebo/Red</material>
+        <mu1>0.8</mu1>
+        <mu2>0.8</mu2>
+        <selfCollide>false</selfCollide>
+      </gazebo>
+    </xacro:if>
   </xacro:macro>
 </robot>
